File: electrical/bionic.kicad_sch (KiCad schematic)
At the start: 36 parts, among them J1 Screw_Terminal_01x04, M1 N20, M2 N20, M3 N20, M4 N20, M5 N20, M6 N20, M7 N20, U1 ESP32, U2 SAMD09, U3 CD4069, U4 CD4069, U5 LM338

Commit message: update(electrical/pcb): Finialized v1.0 Design
Parts:
- added T1: TestPoint_Probe, TestPoint:TestPoint_Pad_1.0x1.0mm, symbol Connector:TestPoint_Probe
- renumbered D5 to D1, D6 to D2, D7 to D3, D8 to D4, D1 to MD1, D2 to MD2, D3 to MD3, D4 to MD4
Connections:
- net +3V3: now also T1.1
Other:
- moved on the sheet: D2
Changed lines of the file:
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@@
 	(wire
 		(pts
-			(xy 106.68 129.54) (xy 93.98 129.54)
+			(xy 93.98 128.27) (xy 81.28 128.27)
 		)
 		(stroke
@@
 	(wire
 		(pts
-			(xy 104.14 123.19) (xy 104.14 127)
+			(xy 91.44 121.92) (xy 91.44 125.73)
 		)
 		(stroke
@@
 	(wire
 		(pts
-			(xy 104.14 127) (xy 93.98 127)
+			(xy 91.44 125.73) (xy 81.28 125.73)
 		)
 		(stroke
@@
 	(wire
 		(pts
-			(xy 101.6 123.19) (xy 101.6 124.46)
+			(xy 88.9 121.92) (xy 88.9 123.19)
 		)
 		(stroke
@@
 	(wire
 		(pts
-			(xy 106.68 129.54) (xy 106.68 123.19)
+			(xy 93.98 128.27) (xy 93.98 121.92)
 		)
 		(stroke
@@
 	(wire
 		(pts
-			(xy 101.6 124.46) (xy 93.98 124.46)
+			(xy 88.9 123.19) (xy 81.28 123.19)
 		)
 		(stroke
@@
 	)
 	(label "+3V3"
-		(at 93.98 127 0)
+		(at 81.28 125.73 0)
 		(fields_autoplaced yes)
 		(effects
@@
 	)
 	(label "+6V"
-		(at 93.98 124.46 0)
+		(at 81.28 123.19 0)
 		(fields_autoplaced yes)
 		(effects
@@
 	)
 	(label "GND"
-		(at 93.98 129.54 0)
+		(at 81.28 128.27 0)
 		(fields_autoplaced yes)
 		(effects
@@
 	)
 	(symbol
+		(lib_id "Connector:TestPoint_Probe")
+		(at 68.58 139.7 90)
+		(unit 1)
+		(exclude_from_sim no)
+		(in_bom yes)
+		(on_board yes)
+		(dnp no)
+		(fields_autoplaced yes)
+		(property "Reference" "T1"
+			(at 66.9925 134.62 90)
+			(effects
+				(font
+					(size 1.27 1.27)
+				)
+			)
+		)
+		(property "Value" "TestPoint_Probe"
+			(at 68.2624 135.89 0)
+			(effects
+				(font
+					(size 1.27 1.27)
+				)
+				(justify left)
+				(hide yes)
+			)
+		)
+		(property "Footprint" "TestPoint:TestPoint_Pad_1.0x1.0mm"
+			(at 68.58 134.62 0)
+			(effects
+				(font
+					(size 1.27 1.27)
+				)
+				(hide yes)
+			)
+		)
+		(property "Datasheet" "~"
+			(at 68.58 134.62 0)
+			(effects
+				(font
+					(size 1.27 1.27)
+				)
+				(hide yes)
+			)
+		)
+		(property "Description" "test point (alternative probe-style design)"
+			(at 68.58 139.7 0)
+			(effects
+				(font
+					(size 1.27 1.27)
+				)
+				(hide yes)
+			)
+		)
+		(pin "1"
+		)
+		(instances
+			(project "bionic"
+				(path "/e63e39d7-6ac0-4ffd-8aa3-1841a4541b55"
+					(reference "T1")
+					(unit 1)
+				)
+			)
+		)
+	)
+	(symbol
 		(lib_id "power:PWR_FLAG")
-		(at 101.6 123.19 0)
+		(at 88.9 121.92 0)
 		(mirror y)
 		(unit 1)
@@
 		(dnp no)
 		(property "Reference" "#FLG02"
-			(at 101.6 121.285 0)
+			(at 88.9 120.015 0)
 			(effects
 				(font
@@
 		)
 		(property "Value" "PWR_FLAG"
-			(at 101.6 119.38 0)
+			(at 88.9 118.11 0)
 			(effects
 				(font
@@
 		)
 		(property "Footprint" ""
-			(at 101.6 123.19 0)
+			(at 88.9 121.92 0)
 			(effects
 				(font
@@
 		)
 		(property "Datasheet" "~"
-			(at 101.6 123.19 0)
+			(at 88.9 121.92 0)
 			(effects
 				(font
@@
 		)
 		(property "Description" "Special symbol for telling ERC where power comes from"
-			(at 101.6 123.19 0)
+			(at 88.9 121.92 0)
 			(effects
 				(font
@@
 		(lib_id "Device:LED_Small")
 		(at 58.42 120.65 0)
-		(mirror x)
 		(unit 1)
 		(exclude_from_sim no)
@@
 		(on_board yes)
 		(dnp no)
-		(property "Reference" "D6"
+		(property "Reference" "D2"
 			(at 58.42 116.84 0)
 			(effects
@@
 		)
 		(property "Value" "LED_Small"
-			(at 58.4835 124.46 0)
+			(at 58.4835 116.84 0)
 			(effects
 				(font
@@
 			(project "bionic"
 				(path "/e63e39d7-6ac0-4ffd-8aa3-1841a4541b55"
-					(reference "D6")
+					(reference "D2")
 					(unit 1)
 				)
@@
 		(dnp no)
 		(fields_autoplaced yes)
-		(property "Reference" "D4"
+		(property "Reference" "MD4"
 			(at 255.27 20.32 0)
 			(effects
@@
 			(project "bionic"
 				(path "/e63e39d7-6ac0-4ffd-8aa3-1841a4541b55"
-					(reference "D4")
+					(reference "MD4")
 					(unit 1)
 				)
@@
 		(on_board yes)
 		(dnp no)
-		(property "Reference" "D8"
+		(property "Reference" "D4"
 			(at 92.71 137.16 0)
 			(effects
@@
 			(project "bionic"
 				(path "/e63e39d7-6ac0-4ffd-8aa3-1841a4541b55"
-					(reference "D8")
+					(reference "D4")
 					(unit 1)
 				)
@@
 		(on_board yes)
 		(dnp no)
-		(property "Reference" "D5"
+		(property "Reference" "D1"
 			(at 46.355 124.46 90)
 			(effects
@@
 			(project "bionic"
 				(path "/e63e39d7-6ac0-4ffd-8aa3-1841a4541b55"
-					(reference "D5")
+					(reference "D1")
 					(unit 1)
 				)
@@
 		(dnp no)
 		(fields_autoplaced yes)
-		(property "Reference" "D1"
+		(property "Reference" "MD1"
 			(at 140.97 20.32 0)
 			(effects
@@
 			(project "bionic"
 				(path "/e63e39d7-6ac0-4ffd-8aa3-1841a4541b55"
-					(reference "D1")
+					(reference "MD1")
 					(unit 1)
 				)
@@
 	(symbol
 		(lib_id "power:PWR_FLAG")
-		(at 104.14 123.19 0)
+		(at 91.44 121.92 0)
 		(mirror y)
 		(unit 1)
@@
 		(dnp no)
 		(property "Reference" "#FLG01"
-			(at 104.14 121.285 0)
+			(at 91.44 120.015 0)
 			(effects
 				(font
@@
 		)
 		(property "Value" "PWR_FLAG"
-			(at 104.14 119.38 0)
+			(at 91.44 118.11 0)
 			(effects
 				(font
@@
 		)
 		(property "Footprint" ""
-			(at 104.14 123.19 0)
+			(at 91.44 121.92 0)
 			(effects
 				(font
@@
 		)
 		(property "Datasheet" "~"
-			(at 104.14 123.19 0)
+			(at 91.44 121.92 0)
 			(effects
 				(font
@@
 		)
 		(property "Description" "Special symbol for telling ERC where power comes from"
-			(at 104.14 123.19 0)
+			(at 91.44 121.92 0)
 			(effects
 				(font
@@
 		(dnp no)
 		(fields_autoplaced yes)
-		(property "Reference" "D2"
+		(property "Reference" "MD2"
 			(at 179.07 20.32 0)
 			(effects
@@
 			(project "bionic"
 				(path "/e63e39d7-6ac0-4ffd-8aa3-1841a4541b55"
-					(reference "D2")
+					(reference "MD2")
 					(unit 1)
 				)
@@
 	(symbol
 		(lib_id "power:PWR_FLAG")
-		(at 106.68 123.19 0)
+		(at 93.98 121.92 0)
 		(mirror y)
 		(unit 1)
@@
 		(dnp no)
 		(property "Reference" "#FLG03"
-			(at 106.68 121.285 0)
+			(at 93.98 120.015 0)
 			(effects
 				(font
@@
 		)
 		(property "Value" "PWR_FLAG"
-			(at 105.41 119.38 0)
+			(at 92.71 118.11 0)
 			(effects
 				(font
@@
 		)
 		(property "Footprint" ""
-			(at 106.68 123.19 0)
+			(at 93.98 121.92 0)
 			(effects
 				(font
@@
 		)
 		(property "Datasheet" "~"
-			(at 106.68 123.19 0)
+			(at 93.98 121.92 0)
 			(effects
 				(font
@@
 		)
 		(property "Description" "Special symbol for telling ERC where power comes from"
-			(at 106.68 123.19 0)
+			(at 93.98 121.92 0)
 			(effects
 				(font
@@
 		(on_board yes)
 		(dnp no)
-		(property "Reference" "D7"
+		(property "Reference" "D3"
 			(at 72.39 143.51 90)
 			(effects
@@
 			(project "bionic"
 				(path "/e63e39d7-6ac0-4ffd-8aa3-1841a4541b55"
-					(reference "D7")
+					(reference "D3")
 					(unit 1)
 				)
@@
 		(dnp no)
 		(fields_autoplaced yes)
-		(property "Reference" "D3"
+		(property "Reference" "MD3"
 			(at 217.17 20.32 0)
 			(effects
@@
 			(project "bionic"
 				(path "/e63e39d7-6ac0-4ffd-8aa3-1841a4541b55"
-					(reference "D3")
+					(reference "MD3")
 					(unit 1)
 				)
